Commit message: update FR5 mass

File: frcobot_description/urdf/fr5_gazebo.urdf (robot description, URDF)
Before this commit: robot fr5_robot, 8 links, 7 joints
Links:
- link base_link: mass 1.073 -> 1.62
- link forearm_Link: mass 20.782 -> 7.67
- link shoulder_Link: mass 4.1676 -> 4.38
- link upperarm_Link: mass 20.782 -> 14.46
- link wrist1_Link: mass 20.782 -> 1.63
- link wrist2_Link: mass 1.570796 -> 1.58
- link wrist3_Link: mass 0.52527 -> 0.53

File: frcobot_description/urdf/fr5_robot.urdf (robot description, URDF)
Before this commit: robot fr5_robot, 8 links, 7 joints
Links:
- link base_link: mass 1.073 -> 1.62
- link forearm_Link: mass 20.782 -> 7.67
- link shoulder_Link: mass 4.1676 -> 4.38
- link upperarm_Link: mass 20.782 -> 14.46
- link wrist1_Link: mass 20.782 -> 1.63
- link wrist2_Link: mass 1.570796 -> 1.58
- link wrist3_Link: mass 0.52527 -> 0.53
