Commit message: update ur10

File: frcobot_description/urdf/fr10_gazebo.urdf (robot description, URDF)
Before this commit: robot FR10-V5.0.SLDASM, 8 links, 7 joints
Links:
- link base_link: mass 0.73773 -> 8.73773
Joints:
- joint j1: origin xyz=0 0 0.045908 rpy=-1.5708 3.14159 3.14159 -> xyz=0 0 0.145908 rpy=-1.5708 3.14159 3.14159
- joint j6: limit lower=-3.0543 upper=3.0543 effort=28 velocity=3.2 -> lower=-3.0543 upper=3.0543 effort=28 velocity=0.2

Commit message: Add camera and color boxes

File: frcobot_description/urdf/fr10_gazebo.urdf (robot description, URDF)
Before this commit: robot FR10-V5.0.SLDASM, 8 links, 7 joints
Links:
- added link realsense_link
Joints:
- added joint realsense_joint: type fixed, parent wrist3_Link, child realsense_link, origin xyz=0 0.3 0 rpy=0 0 1.57

File: frcobot_description/urdf/fr3_gazebo.urdf (robot description, URDF)
Before this commit: robot FR3-V5.0, 8 links, 7 joints
Links:
- added link realsense_link
Joints:
- added joint realsense_joint: type fixed, parent wrist3_Link, child realsense_link, origin xyz=0 0.1 0 rpy=-1.57 0 1.57

Commit message: Update gazebo control

File: frcobot_description/urdf/fr10_gazebo.urdf (robot description, URDF)
Before this commit: robot FR10-V5.0.SLDASM, 9 links, 8 joints
Links:
- link realsense_link: mass None -> 0.14186
Joints:
- joint j1: origin xyz=0 0 0.145908 rpy=-1.5708 3.14159 3.14159 -> xyz=0 0 0.045908 rpy=-1.5708 3.14159 3.14159

File: gazebo_ros_model_color/urdf/box.gazebo.urdf.xacro (robot description, xacro)
@@ -2,9 +2,62 @@
 <robot name="color_box">
   <link name="world"/>
-  <joint name="world_box_joint" type="fixed">
-    <parent link="world"/>
-    <child link="my_color_box"/>
-  </joint>
-  <link name="my_color_box">
+  <link name="my_color_box1">
+    <inertial>
+      <origin xyz="0 0 0" />
+      <mass value="1.0" />
+    <inertia  ixx="1.0" ixy="0.0"  ixz="0.0"  iyy="100.0"  iyz="0.0"  izz="1.0" />
+    </inertial>
+    <visual>
+      <origin xyz="0 0 0"/>
+      <geometry>
+        <box size="0.5 0.5 0.5" />
+      </geometry>
+    </visual>
+    <collision>
+      <origin xyz="0 0 0"/>
+      <geometry>
+        <box size="0.5 0.5 0.5" />
+      </geometry>
+    </collision>
+  </link>
+  <link name="my_color_box2">
+    <inertial>
+      <origin xyz="0 0 0" />
+      <mass value="1.0" />
+    <inertia  ixx="1.0" ixy="0.0"  ixz="0.0"  iyy="100.0"  iyz="0.0"  izz="1.0" />
+    </inertial>
+    <visual>
+      <origin xyz="0 0 0"/>
+      <geometry>
+        <box size="0.5 0.5 0.5" />
+      </geometry>
+    </visual>
+    <collision>
+      <origin xyz="0 0 0"/>
+      <geometry>
+        <box size="0.5 0.5 0.5" />
+      </geometry>
+    </collision>
+  </link>
+  <link name="my_color_box3">
+    <inertial>
+      <origin xyz="0 0 0" />
+      <mass value="1.0" />
+    <inertia  ixx="1.0" ixy="0.0"  ixz="0.0"  iyy="100.0"  iyz="0.0"  izz="1.0" />
+    </inertial>
+    <visual>
+      <origin xyz="0 0 1"/>
+      <geometry>
+        <box size="0.5 0.5 0.5" />
+      </geometry>
+    </visual>
+    <collision>
+      <origin xyz="0 0 0"/>
+      <geometry>
+        <box size="0.5 0.5 0.5" />
+      </geometry>
+    </collision>
+  </link>
+  <link name="my_color_box4">
     <inertial>
       <origin xyz="2 0 0" />
@@ -13,5 +66,5 @@
     </inertial>
     <visual>
-      <origin xyz="2 0 1"/>
+      <origin xyz="2 0 0"/>
       <geometry>
         <box size="0.5 0.5 0.5" />
@@ -19,5 +72,5 @@
     </visual>
     <collision>
-      <origin xyz="2 0 1"/>
+      <origin xyz="2 0 0"/>
       <geometry>
         <box size="0.5 0.5 0.5" />
@@ -25,12 +78,62 @@
     </collision>
   </link>
-  <gazebo reference='my_color_box'>
+  <link name="my_color_box5">
+    <inertial>
+      <origin xyz="0 0 0" />
+      <mass value="1.0" />
+    <inertia  ixx="1.0" ixy="0.0"  ixz="0.0"  iyy="100.0"  iyz="0.0"  izz="1.0" />
+    </inertial>
     <visual>
-      <plugin name="gazebo_ros_model_color" filename="libgazebo_ros_model_color.so">
-        <robotNamespace>/</robotNamespace>
-        <serviceName>/my_box_color</serviceName>
-        <color>0.5 0.8 1.0 1.0</color>
-      </plugin>
+      <origin xyz="0 0 0"/>
+      <geometry>
+        <box size="0.5 0.5 0.5" />
+      </geometry>
     </visual>
+    <collision>
+      <origin xyz="0 0 0"/>
+      <geometry>
+        <box size="0.5 0.5 0.5" />
+      </geometry>
+    </collision>
+  </link>
+  <joint name="world_box_joint1" type="fixed">
+    <origin xyz="3 0 1" />
+    <parent link="world"/>
+    <child link="my_color_box1"/>
+  </joint>
+  <joint name="world_box_joint2" type="fixed">
+    <origin xyz="-2 0 1" />
+    <parent link="world"/>
+    <child link="my_color_box2"/>
+  </joint>
+  <joint name="world_box_joint3" type="fixed">
+    <origin xyz="-2 -2 1" />
+    <parent link="world"/>
+    <child link="my_color_box3"/>
+  </joint>
+  <joint name="world_box_joint4" type="fixed">
+    <origin xyz="2 2 1" />
+    <parent link="world"/>
+    <child link="my_color_box4"/>
+  </joint>
+  <joint name="world_box_joint5" type="fixed">
+    <origin xyz="0 -2 1"/>
+    <parent link="world"/>
+    <child link="my_color_box5"/>
+  </joint>
+  <gazebo reference='my_color_box1'>
+    <material value="Gazebo/Blue"/>
+  </gazebo>
+  <gazebo reference='my_color_box2'>
+    <material value="Gazebo/Red"/>
+  </gazebo>
+  <gazebo reference='my_color_box3'>
+    <material value="Gazebo/Green"/>
+  </gazebo>
+  <gazebo reference='my_color_box4'>
+    <material value="Gazebo/Grey"/>
+  </gazebo>
+  <gazebo reference='my_color_box5'>
+    <material value="Gazebo/Yellow"/>
   </gazebo>
 </robot>

Commit message: Add gripper

File: frcobot_description/urdf/fr10_gazebo.urdf (robot description, URDF)
Before this commit: robot FR10-V5.0.SLDASM, 9 links, 8 joints
Links:
- added link rh_p12_rn_base, mass 0.236; collision mesh filename=package://husky_ur3_gazebo/meshes/base.stl scale=0.001 0.001 0.001; visual mesh filename=package://husky_ur3_gazebo/meshes/base.stl scale=0.001 0.001 0.001
- added link rh_p12_rn_l1, mass 0.068; visual mesh filename=package://husky_ur3_gazebo/meshes/l1.stl scale=0.001 0.001 0.001
- added link rh_p12_rn_l2, mass 0.0022; collision mesh filename=package://husky_ur3_gazebo/meshes/l2.stl scale=0.001 0.001 0.001; visual mesh filename=package://husky_ur3_gazebo/meshes/l2.stl scale=0.001 0.001 0.001
- added link rh_p12_rn_r1, mass 0.068; visual mesh filename=package://husky_ur3_gazebo/meshes/r1.stl scale=0.001 0.001 0.001
- added link rh_p12_rn_r2, mass 0.0022; collision mesh filename=package://husky_ur3_gazebo/meshes/r2.stl scale=0.001 0.001 0.001; visual mesh filename=package://husky_ur3_gazebo/meshes/r2.stl scale=0.001 0.001 0.001
Joints:
- added joint rh_l1: type revolute, parent rh_p12_rn_base, child rh_p12_rn_l1, origin xyz=0.0 -0.008 0.048 rpy=0 0 0, axis -1 0 0, limit lower=-3.0543 upper=3.0543 effort=28 velocity=0.002
- added joint rh_l2: type fixed, parent rh_p12_rn_l1, child rh_p12_rn_l2, origin xyz=0.0 -0.0493634 0.0285 rpy=0 0 0, axis 1 0 0, limit lower=-3.0543 upper=3.0543 effort=28 velocity=0.002
- added joint rh_p12_rn: type revolute, parent rh_p12_rn_base, child rh_p12_rn_r1, origin xyz=0.0 0.008 0.048 rpy=0 0 0, axis 1 0 0, limit lower=-3.0543 upper=3.0543 effort=28 velocity=0.002
- added joint rh_r2: type fixed, parent rh_p12_rn_r1, child rh_p12_rn_r2, origin xyz=0.0 0.0493634 0.0285 rpy=0 0 0, axis -1 0 0, limit lower=-3.0543 upper=3.0543 effort=28 velocity=0.002
- added joint ur3_gripper_joint: type fixed, parent wrist3_Link, child rh_p12_rn_base, origin xyz=0 0.05 0 rpy=-1.57 0 0
- joint j6: origin xyz=-0.060457 -0.0602 -0.0046473 rpy=-3.1416 2.54 0 -> xyz=-0.060457 -0.0602 -0.0046473 rpy=-3.1416 0 0

Commit message: add meshes

File: frcobot_description/urdf/fr10_gazebo.urdf (robot description, URDF)
Before this commit: robot FR10-V5.0.SLDASM, 14 links, 13 joints
Links:
- link rh_p12_rn_base: geometry collision mesh filename=package://frcobot_description/meshes/gripper//base.stl scale=0.001 0.001 0.001; visual mesh filename=package://frcobot_description/meshes/gripper//base.stl scale=0.001 0.001 0.001
- link rh_p12_rn_l1: geometry visual mesh filename=package://frcobot_description/meshes/gripper//l1.stl scale=0.001 0.001 0.001
- link rh_p12_rn_l2: geometry collision mesh filename=package://frcobot_description/meshes/gripper//l2.stl scale=0.001 0.001 0.001; visual mesh filename=package://frcobot_description/meshes/gripper//l2.stl scale=0.001 0.001 0.001
- link rh_p12_rn_r1: geometry visual mesh filename=package://frcobot_description/meshes/gripper//r1.stl scale=0.001 0.001 0.001
- link rh_p12_rn_r2: geometry collision mesh filename=package://frcobot_description/meshes/gripper//r2.stl scale=0.001 0.001 0.001; visual mesh filename=package://frcobot_description/meshes/gripper//r2.stl scale=0.001 0.001 0.001

Commit message: update task code

File: frcobot_description/urdf/fr10_gazebo.urdf (robot description, URDF)
Before this commit: robot FR10-V5.0.SLDASM, 14 links, 13 joints
Links:
- added link rh_p12_rn_tf_end, mass 0.01
- link realsense_link: geometry collision box size=0.02 0.1 0.04; visual box size=0.02 0.1 0.04
Joints:
- added joint rh_p12_rn_tf: type fixed, parent wrist3_Link, child rh_p12_rn_tf_end, origin xyz=0.0 0.15 0.0 rpy=-1.57 0 1.57
- joint realsense_joint: origin xyz=0 0.3 0 rpy=0 0 1.57 -> xyz=-0.06 0.08 0 rpy=-1.57 0 1.57

Commit message: stable task_executer

File: frcobot_description/urdf/fr10_gazebo.urdf (robot description, URDF)
Before this commit: robot FR10-V5.0.SLDASM, 15 links, 14 joints
Links:
- added link ground_plane_box; collision box size=10.0 10.0 0.005; visual box size=10.0 10.0 0.005
Joints:
- added joint ground_plane_box: type fixed, parent world, child ground_plane_box, origin xyz=0 0 -0.005 rpy=0 0 0

File: frcobot_description/urdf/fr3_gazebo.urdf (robot description, URDF)
Before this commit: robot FR3-V5.0, 9 links, 8 joints
Links:
- added link ground_plane_box; collision box size=10.0 10.0 0.005; visual box size=10.0 10.0 0.005
Joints:
- added joint ground_plane_box: type fixed, parent world, child ground_plane_box, origin xyz=0 0 -0.0025 rpy=0 0 0

Commit message: add octomap

File: frcobot_description/urdf/fr10_gazebo.urdf (robot description, URDF)
Before this commit: robot FR10-V5.0.SLDASM, 16 links, 15 joints
Links:
- added link realsense_phantom_link, mass 0.001
Joints:
- added joint realsense_phantom_joint: type fixed, parent wrist3_Link, child realsense_phantom_link, origin xyz=-0.06 0.08 0 rpy=-1.57 -1.57 0

File: frcobot_description/urdf/fr3_gazebo.urdf (robot description, URDF)
Before this commit: robot FR3-V5.0, 10 links, 9 joints
Links:
- added link realsense_phantom_link, mass 0.001
Joints:
- added joint realsense_phantom_joint: type fixed, parent wrist3_Link, child realsense_phantom_link, origin xyz=-0.06 0.08 0 rpy=-1.57 -1.57 0

Commit message: stable moveit_python

File: frcobot_description/urdf/fr10_gazebo.urdf (robot description, URDF)
Before this commit: robot FR10-V5.0.SLDASM, 17 links, 16 joints
Links:
- removed link rh_p12_rn_tf_end
- added link tf_end, mass 0.01
Joints:
- removed joint rh_p12_rn_tf
- added joint r_tf_end: type fixed, parent wrist3_Link, child tf_end, origin xyz=0.0 0.15 0.0 rpy=-1.57 0 1.57
- joint j6: limit lower=-3.0543 upper=3.0543 effort=28 velocity=0.2 -> lower=-3.0543 upper=3.0543 effort=28 velocity=4.0

File: frcobot_description/urdf/fr10_robot.urdf (robot description, URDF)
Before this commit: robot FR10-V5.0.SLDASM, 8 links, 7 joints
Links:
- added link tf_end, mass 0.01
Joints:
- added joint r_tf_end: type fixed, parent wrist3_Link, child tf_end, origin xyz=0.0 0.15 0.0 rpy=-1.57 0 1.57

File: frcobot_description/urdf/fr3_gazebo.urdf (robot description, URDF)
Before this commit: robot FR3-V5.0, 11 links, 10 joints
Links:
- added link tf_end, mass 0.01
Joints:
- added joint r_tf_end: type fixed, parent wrist3_Link, child tf_end, origin xyz=0.0 0.15 0.0 rpy=-1.57 0 1.57

File: frcobot_description/urdf/fr3_robot.urdf (robot description, URDF)
Before this commit: robot FR3-V5.0, 8 links, 7 joints
Links:
- added link tf_end, mass 0.01
Joints:
- added joint r_tf_end: type fixed, parent wrist3_Link, child tf_end, origin xyz=0.0 0.15 0.0 rpy=-1.57 0 1.57
